Commit message: Ongoing : tf error fixing for gmapping

File: lio_sam/launch/include/config/robot.urdf.xacro (robot description, xacro)
@@ -10,9 +10,9 @@
   </joint>
   <link name="imu_link"> </link>
-  <joint name="imu_joint" type="fixed">
+  <!-- <joint name="imu_joint" type="fixed">
     <parent link="chassis_link" />
     <child link="imu_link" />
     <origin xyz="0 0 0" rpy="0 0 0" />
-  </joint>
+  </joint> -->
   <link name="velodyne"> </link>
   <joint name="velodyne_joint" type="fixed">

Commit message: Fix : two root links

File: lio_sam/launch/include/config/robot.urdf.xacro (robot description, xacro)
@@ -9,5 +9,5 @@
     <origin xyz="0 0 0" rpy="0 0 0" />
   </joint>
-  <link name="imu_link"> </link>
+  <!-- <link name="imu_link"> </link> -->
   <!-- <joint name="imu_joint" type="fixed">
     <parent link="chassis_link" />
